File: bjt-push-pull/bjt-push-pull.kicad_sch (KiCad schematic)
At the start: 11 parts, among them Q1 2N3904, Q2 2N3906, Q3 2N3904, Q4 2N3906

Commit message: bugfix: use local spice file
Parts:
- Q1, Q3, Q4: Spice_Lib_File /usr/home/trombik/github/KiCad-Spice-Library/Models/Transis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 -> BJT.lib
- Q2: Spice_Lib_File /home/trombik/github/KiCad-Spice-Library/Models/Transistor/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 -> BJT.lib
Changed lines of the file:
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@@
       (effects (font (size 1.27 1.27)) hide)
     )
-    (property "Spice_Lib_File" "/usr/home/trombik/github/KiCad-Spice-Library/Models/Transistor/BJT/BJT.lib" (id 7) (at 113.03 76.2 0)
+    (property "Spice_Lib_File" "BJT.lib" (id 7) (at 113.03 76.2 0)
       (effects (font (size 1.27 1.27)) hide)
     )
@@
       (effects (font (size 1.27 1.27)) hide)
     )
-    (property "Spice_Lib_File" "/home/trombik/github/KiCad-Spice-Library/Models/Transistor/BJT/BJT.lib" (id 7) (at 113.03 92.71 0)
+    (property "Spice_Lib_File" "BJT.lib" (id 7) (at 113.03 92.71 0)
       (effects (font (size 1.27 1.27)) hide)
     )
@@
       (effects (font (size 1.27 1.27)) hide)
     )
-    (property "Spice_Lib_File" "/usr/home/trombik/github/KiCad-Spice-Library/Models/Transistor/BJT/BJT.lib" (id 7) (at 125.73 76.2 0)
+    (property "Spice_Lib_File" "BJT.lib" (id 7) (at 125.73 76.2 0)
       (effects (font (size 1.27 1.27)) hide)
     )
@@
       (effects (font (size 1.27 1.27)) hide)
     )
-    (property "Spice_Lib_File" "/usr/home/trombik/github/KiCad-Spice-Library/Models/Transistor/BJT/BJT.lib" (id 7) (at 125.73 92.71 0)
-      (effects (font (size 1.27 1.27)) hide)
-    )
+    (property "Spice_Lib_File" "BJT.lib" (id 7) (at 125.73 92.71 0)
+      (effects (font (size 1.27 1.27)) hide)
+    )
